File: pcb/new pcb/new pcb.kicad_sch (KiCad schematic)
At the start: 42 parts, among them J1 Lidar conector, J10 Conn_01x04, J11 Conn_01x04, J12 Conn_01x04, J13 Conn_01x04, J14 Conn_01x04, J15 Conn_01x04, J2 RJ9, J3 I2C quiic conector, J5 Conn_01x04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

Commit message: fix the pcb
Parts:
- added R12, R13: 100, Resistor_SMD:R_1206_3216Metric_Pad1.30x1.75mm_HandSolder, symbol Device:R
Connections:
- net GND: now also R12.2, R13.1
- net at A1.D1 (SWCLK): now also debug1.1 (Pin_1), R12.1; no longer debug1.3 (Pin_3)
- net at A1.D3 (SWDIO): now also debug1.3 (Pin_3), R13.2; no longer debug1.1 (Pin_1)

Commit message: actual fix
Parts:
- removed R12, R13: 100, Resistor_SMD:R_1206_3216Metric_Pad1.30x1.75mm_HandSolder, symbol Device:R

Commit message: added reset to gpio14
Connections:
- net at A1.19 (GPIO14): now also U3.3 (~{RESET})
Changed lines of the file:
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@@
+	(wire
+		(pts
+			(xy 153.67 97.79) (xy 153.67 113.03)
+		)
+		(stroke
+			(width 0)
+			(type default)
+		)
+	)
 	(wire
 		(pts
@@
 	(wire
 		(pts
+			(xy 50.8 113.03) (xy 50.8 147.32)
+		)
+		(stroke
+			(width 0)
+			(type default)
+		)
+	)
+	(wire
+		(pts
 			(xy 107.95 173.99) (xy 111.76 173.99)
 		)
@@
 	(wire
 		(pts
+			(xy 176.53 97.79) (xy 153.67 97.79)
+		)
+		(stroke
+			(width 0)
+			(type default)
+		)
+	)
+	(wire
+		(pts
 			(xy 152.4 82.55) (xy 166.37 82.55)
 		)
@@
 	(wire
 		(pts
+			(xy 153.67 113.03) (xy 50.8 113.03)
+		)
+		(stroke
+			(width 0)
+			(type default)
+		)
+	)
+	(wire
+		(pts
 			(xy 175.26 67.31) (xy 176.53 67.31)
 		)
@@
 		)
 		(stroke
+			(width 0)
+			(type default)
+		)
+	)
+	(wire
+		(pts
+			(xy 50.8 147.32) (xy 53.34 147.32)
+		)
+		(stroke
